Commit message: See low objects and all round: LiDAR in the costmaps, 5 cm band, 5 cm margin
The owner asked for wires, remotes and 6-8 cm objects to be seen, for a 5 cm
safety margin, and for safe turns at corners.

- The LiDAR is in both nav2 costmaps (ObstacleLayer on /scan). Until now both
  were camera-only: nav2 knew nothing beside or behind the rover. Live, the
  local costmap now holds 1043 lethal cells behind the rover.
- nvblox's obstacle band is now 5-27 cm (was 10-24). The 10 cm floor existed
  because the TF called the camera level while it was not, so the floor rose
  with range. New `./rover camera --floor` measures the tilt off the floor in
  the camera's own depth (RANSAC over ~40k points, 3.5 mm rms, two runs): roll
  -1.4 deg, pitch ~0, height 0.172 (tape 0.175). The old "-1.3 deg pitch" was
  a gravity reading from an older mount at 16.3 cm. With the tilt in the TF,
  bare floor 0.4-1.3 m ahead reads 97% within -5..+4 cm and nvblox marks
  none of it. The top of the band is the LiDAR puck's top, 26.1 cm.
- vo_node now uses the full base_link -> camera0_link rotation from TF, not
  only its translation; its self-test passes.
- footprint_padding 0.05 (was 0.03), as asked. RPP and the Spin recovery sweep
  the padded footprint as it rotates. The real pivot still slides ~30 cm per
  90 deg, so ./rover drive still plans turns.

floor_calib's plane fit first ran out of memory: a full SVD built a 24k x 24k
matrix. It now uses the 3x3 covariance.

Co-Authored-By: Claude Opus 5.5 <noreply@anthropic.com>

File: description/rover.urdf (robot description, URDF)
Before this commit: robot rover, 10 links, 9 joints
Joints:
- joint camera_joint: origin xyz=0.173 -0.0475 0.175 rpy=0 0 0 -> xyz=0.173 -0.0475 0.175 rpy=-0.0245 0 0

Commit message: Camera lever arm fitted against LiDAR truth: the left imager is on the LEFT
Stage A's baseline is now recorded: pivot90 (6 of 8 turns), pivot360, a
single turn, and a 0.4 m square, on the charged pack. After every turn,
fused and VO were ~13 cm off even when the rover barely moved: a lever-arm
error. Re-projecting the recorded VO with candidate camera offsets against
LiDAR truth (26 checkpoints, 7 runs) fits camera0_link at
(0.1623, +0.0419) +- 3 mm. The mean error drops from 8.0 to 2.0 cm and the
max from 19.6 to 5.7. Leave-one-run-out holds (e.g. held-out 13.6 -> 1.3 cm).

The D555 driver's TF sign put the left imager on the right. The old y = 0
explains TODO 43's "7 cm per turn" (0.0475 * sqrt 2). params.yaml gains
vo_lever_x/y (calibrated) and infra2_side -1. The URDF and vo_node's
fallback follow, and the fit is live.

Also:
- the gyro under-reads turns by ~2% (363 vs 369.7 deg over four turns)
- the pivot slide varies, 6-22 cm per 90 on a charged pack
- one turn froze with a healthy link, which fits BTS7960 protection
- harness: a `turn` scenario; turn clearance checks the exact swept outline
  plus the 5 cm margin instead of a full circle; self-filter for returns
  inside the rover
- pivot_goto and pivot_test get the same self-filter: something on the
  rear-right corner reaches the laser plane

Co-Authored-By: Claude Opus 5.5 <noreply@anthropic.com>

File: description/rover.urdf (robot description, URDF)
Before this commit: robot rover, 10 links, 9 joints
Joints:
- joint camera_joint: origin xyz=0.173 -0.0475 0.175 rpy=-0.0245 0 0 -> xyz=0.1623 0.0419 0.175 rpy=-0.0245 0 0

Commit message: M1: camera yaw measured against the LiDAR, now the only camera yaw
`./rover camera --lidar` from 6 hand-placed poses facing corners. Per spot:
+1.59 -0.29 +0.71 +1.13 +0.98 +1.57 deg, median +0.96. The depth scale fits
at 1.00; +-3% moves the residual under 0.1 cm.

- params.yaml camera.yaw 0.0168 rad (0.96 deg), in the URDF. Depth, nvblox
  and the costmaps all follow it.
- vo_node takes roll, pitch and yaw from TF. cam_yaw_deg is now an EXTRA
  correction (default 0). The August 2.06 deg came from an older mount, and
  it fit LiDAR truth worst of the values tried (mean 2.03 cm vs 1.75 at
  0.96). It is kept only for the self-test.
- Independent check: the same fits put camera0_link within 4 mm of the VO
  lever-arm fit (0.162, +0.046 vs 0.1623, +0.0419).
- The solver takes the median; residual weighting let two tight poses and an
  outlier drag the answer to +0.45. Captures average 45 depth frames and 60
  scans.
- Limit, stated: at one unmoved spot the remaining correction reads
  +0.5..+0.95 while other spots sit near 0. The angle varies by scene, so
  ~1.0 +- 0.3 deg is what this method can prove.

Co-Authored-By: Claude Opus 5.5 <noreply@anthropic.com>

File: description/rover.urdf (robot description, URDF)
Before this commit: robot rover, 10 links, 9 joints
Joints:
- joint camera_joint: origin xyz=0.1623 0.0419 0.175 rpy=-0.0245 0 0 -> xyz=0.1623 0.0419 0.175 rpy=-0.0245 0 0.0168

Commit message: Camera tilt re-measured: pitch +0.50, roll -0.85 deg (was 0.0 / -1.40)
./rover camera --floor on clear floor, 2026-09-28 after a power cycle and
the rover being lifted by hand: 73% of 40k points on the plane, 3.3 mm rms.
The 0.5 deg of pitch the TF did not know made the floor rise ~2.6 cm by
3 m; with depth noise, far floor crossed nvblox 5 cm obstacle band. After
applying it (description/build, lidar..vlm restarted): ghost_check shows 0
camera-only cells from 0.35 to 1.35 m on the same clear floor.

Co-Authored-By: Claude Opus 5.5 <noreply@anthropic.com>

File: description/rover.urdf (robot description, URDF)
Before this commit: robot rover, 10 links, 9 joints
Joints:
- joint camera_joint: origin xyz=0.1623 0.0419 0.175 rpy=-0.0245 0 0.0168 -> xyz=0.1623 0.0419 0.175 rpy=-0.0149 0.0086 0.0168

Commit message: Camera re-calibrated: pitch 0.49 -> 3.02 deg (the mount moved); fake red on the glossy floor before the door
ghost_check before: 1913 camera-only lethal cells 0.85-1.85 m ahead, LiDAR none.
Three ./rover camera --floor runs agree (2.93-3.07 deg, 84% on plane, 3 mm rms).
After: 497, the open floor ahead clean.

Co-Authored-By: Claude Opus 5.5 <noreply@anthropic.com>

File: description/rover.urdf (robot description, URDF)
Before this commit: robot rover, 10 links, 9 joints
Joints:
- joint camera_joint: origin xyz=0.1623 0.0419 0.175 rpy=-0.0149 0.0086 0.0168 -> xyz=0.1623 0.0419 0.175 rpy=-0.0025 0.0528 0.0168

Commit message: description: the two front sonars -- params, frames sonar_left / sonar_right
Owner, 2026-10-19: two HC-SR04-type sensors (run at 3.3 V) at the front
corners, each centre 6.5 cm above the floor, 28 cm apart (the frame's
width), on their own ESP32. Bench-tested: a flat target at 15 cm read
14.4-15.5 / 15.0 cm.

params.yaml `sonar`: z, spacing (described); face_inset, yaw_out, pitch_up
and which one is left (S1 = TRIG GPIO5) are ASSUMED (flush, straight, level,
S1 left) -- listed on every build until measured; fov 0.26 rad, 0.02-4.0 m
(datasheet). build.py: frames sonar_left (0.182, +0.14, 0.065) and
sonar_right (0.182, -0.14, 0.065), x along the beam -- what /sonar/left and
/sonar/right (sensor_msgs/Range) will be stamped in, here and in the twin.

Co-Authored-By: Claude Opus 5.5 <noreply@anthropic.com>

File: description/rover.urdf (robot description, URDF)
Before this commit: robot rover, 10 links, 9 joints
Links:
- added link sonar_left; collision box size=0.02 0.045 0.02; visual box size=0.02 0.045 0.02
- added link sonar_right; collision box size=0.02 0.045 0.02; visual box size=0.02 0.045 0.02
Joints:
- added joint sonar_left_joint: type fixed, parent base_link, child sonar_left, origin xyz=0.182 0.14 0.065 rpy=0 0 0
- added joint sonar_right_joint: type fixed, parent base_link, child sonar_right, origin xyz=0.182 -0.14 0.065 rpy=0 0 0
